File: RelayModule/RelayModule.kicad_pcb (KiCad board)
At the start: 2 copper layers, 49.9 x 21.3 mm, 16 parts, among them P1 Control_connector, P2 Power_connector, Q1 S8050, U1 PC817

Commit message: logo atomo añadido
Parts:
- removed the G*** at (175.3, 99.7)
- added G***: LOGO, Grape:atom_small, B.Cu at (152.3, 106.4)
- G***: moved to B.Cu
- moved G*** 1.28 mm to (173.1, 108.6), turned to 180 degrees
Routing:
- added copper zone on B.Cu, net GND
- added copper zone on F.Cu, net GND

Commit message: Conector cambiado
Routing:
- net GND: track 38.0 -> 11.3 mm, vias 1 -> 0
- net VCC: track 28.7 -> 37.4 mm, vias 0 -> 1
- net Net-(R2-Pad1): track 11.8 -> 11.0 mm, vias 0 -> 1
Changed lines of the file:
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@@
     (area 148.145499 88.963499 198.184295 110.427295)
     (thickness 1.6)
-    (drawings 32)
-    (tracks 79)
+    (drawings 34)
+    (tracks 77)
     (zones 0)
     (modules 16)
@@
   )
   (module Connectors_JST:JST_PH_S3B-PH-K_03x2.00mm_Angled (layer F.Cu)
-    (at 150.622 97.663 270)
+    (at 150.622 97.6376 270)
     (descr http://www.jst-mfg.com/product/pdf/eng/ePH.pdf)
     (tags "connector jst ph")
@@
       (xy -0.810544 2.875975) (xy -0.751292 2.887789) (xy -0.692601 2.887765)) (layer B.Mask) (width 0.01))
   )
+  (gr_line (start 151.9936 95.7072) (end 142.8496 95.7072) (angle 90) (layer Dwgs.User) (width 0.127))
+  (gr_line (start 151.9936 95.8088) (end 151.9936 78.6384) (angle 90) (layer Dwgs.User) (width 0.127))
   (dimension 25.019 (width 0.127) (layer Dwgs.User)
     (gr_text "25,019 mm" (at 160.5915 80.5355) (layer Dwgs.User)
@@
   (segment (start 150.942 91.882) (end 150.792 92.032) (width 0.3) (layer F.Cu) (net 1))
   (segment (start 150.792 92.032) (end 150.792 93.726) (width 0.4) (layer F.Cu) (net 1))
-  (segment (start 155.514 106.188) (end 155.514 106.873) (width 0.254) (layer F.Cu) (net 2))
-  (segment (start 151.892 96.393) (end 150.622 97.663) (width 0.254) (layer B.Cu) (net 2))
-  (segment (start 156.591 96.393) (end 151.892 96.393) (width 0.254) (layer B.Cu) (net 2))
-  (segment (start 157.353 95.631) (end 156.591 96.393) (width 0.254) (layer B.Cu) (net 2))
-  (segment (start 157.353 92.456) (end 157.353 95.631) (width 0.254) (layer B.Cu) (net 2))
-  (segment (start 157.861 91.948) (end 157.353 92.456) (width 0.254) (layer B.Cu) (net 2))
-  (segment (start 159.385 91.948) (end 157.861 91.948) (width 0.254) (layer B.Cu) (net 2))
-  (segment (start 159.893 92.456) (end 159.385 91.948) (width 0.254) (layer B.Cu) (net 2))
-  (segment (start 159.893 105.156) (end 159.893 92.456) (width 0.254) (layer B.Cu) (net 2))
-  (segment (start 159.131 105.918) (end 159.893 105.156) (width 0.254) (layer B.Cu) (net 2))
-  (via (at 159.131 105.918) (size 0.6858) (drill 0.3302) (layers F.Cu B.Cu) (net 2))
-  (segment (start 159.131 106.045) (end 159.131 105.918) (width 0.254) (layer F.Cu) (net 2))
-  (segment (start 157.988 107.188) (end 159.131 106.045) (width 0.254) (layer F.Cu) (net 2))
-  (segment (start 155.829 107.188) (end 157.988 107.188) (width 0.254) (layer F.Cu) (net 2))
-  (segment (start 155.514 106.873) (end 155.829 107.188) (width 0.254) (layer F.Cu) (net 2))
-  (segment (start 152.992 93.726) (end 152.992 95.166) (width 0.4) (layer F.Cu) (net 2))
-  (segment (start 150.622 96.774) (end 150.622 97.79) (width 0.4) (layer F.Cu) (net 2))
-  (segment (start 151.13 96.266) (end 150.622 96.774) (width 0.4) (layer F.Cu) (net 2))
-  (segment (start 151.892 96.266) (end 151.13 96.266) (width 0.4) (layer F.Cu) (net 2))
-  (segment (start 152.992 95.166) (end 151.892 96.266) (width 0.4) (layer F.Cu) (net 2))
+  (segment (start 155.514 106.188) (end 155.3116 106.188) (width 0.254) (layer F.Cu) (net 2) (status C00000))
+  (segment (start 155.3116 106.188) (end 154.5336 105.41) (width 0.254) (layer F.Cu) (net 2) (status 400000))
+  (segment (start 154.5336 105.41) (end 154.5336 104.0892) (width 0.254) (layer F.Cu) (net 2))
+  (segment (start 154.5336 104.0892) (end 152.9588 102.5144) (width 0.254) (layer F.Cu) (net 2))
+  (segment (start 152.9588 102.5144) (end 152.5524 102.5144) (width 0.254) (layer F.Cu) (net 2))
+  (segment (start 152.5524 102.5144) (end 152.3492 102.3112) (width 0.254) (layer F.Cu) (net 2))
+  (segment (start 152.3492 102.3112) (end 152.3492 98.806) (width 0.254) (layer F.Cu) (net 2))
+  (segment (start 152.3492 98.806) (end 151.1808 97.6376) (width 0.254) (layer F.Cu) (net 2) (status 800000))
+  (segment (start 151.1808 97.6376) (end 150.622 97.6376) (width 0.254) (layer F.Cu) (net 2) (status C00000))
   (segment (start 154.178 100.838) (end 154.178 102.87) (width 0.5) (layer B.Cu) (net 3))
   (segment (start 153.246 104.31) (end 153.246 105.41) (width 0.5) (layer F.Cu) (net 3))
@@
   (segment (start 153.289 103.759) (end 153.289 104.267) (width 0.5) (layer B.Cu) (net 3))
   (segment (start 154.178 102.87) (end 153.289 103.759) (width 0.5) (layer B.Cu) (net 3))
-  (segment (start 151.046 105.41) (end 151.046 102.214) (width 0.4) (layer F.Cu) (net 4))
-  (segment (start 151.046 102.214) (end 150.622 101.79) (width 0.3) (layer F.Cu) (net 4))
+  (segment (start 151.046 105.41) (end 151.046 104.31) (width 0.254) (layer F.Cu) (net 4))
+  (segment (start 150.622 103.886) (end 150.622 101.6376) (width 0.254) (layer F.Cu) (net 4))
+  (segment (start 151.046 104.31) (end 150.622 103.886) (width 0.254) (layer F.Cu) (net 4))
   (segment (start 161.798 98.298) (end 161.798 97.662) (width 0.5) (layer F.Cu) (net 5))
   (segment (start 161.798 97.662) (end 158.75 94.614) (width 0.5) (layer F.Cu) (net 5))
@@
   (segment (start 161.082 105.364) (end 168.32 105.364) (width 0.4) (layer F.Cu) (net 6))
   (segment (start 158.258 108.188) (end 161.082 105.364) (width 0.4) (layer F.Cu) (net 6))
+  (segment (start 152.842 91.44) (end 152.908 91.44) (width 0.254) (layer F.Cu) (net 7))
+  (segment (start 152.908 91.44) (end 153.7208 92.2528) (width 0.254) (layer F.Cu) (net 7))
+  (segment (start 151.924 99.6376) (end 150.622 99.6376) (width 0.254) (layer B.Cu) (net 7))
+  (segment (start 152.6032 98.9584) (end 151.924 99.6376) (width 0.254) (layer B.Cu) (net 7))
+  (segment (start 152.6032 93.3704) (end 152.6032 98.9584) (width 0.254) (layer B.Cu) (net 7))
+  (segment (start 153.7208 92.2528) (end 152.6032 93.3704) (width 0.254) (layer B.Cu) (net 7))
+  (via (at 153.7208 92.2528) (size 0.6858) (drill 0.3302) (layers F.Cu B.Cu) (net 7))
   (segment (start 149.098 100.838) (end 149.098 90.678) (width 0.4) (layer F.Cu) (net 7))
   (segment (start 152.842 90.739) (end 152.842 91.44) (width 0.4) (layer F.Cu) (net 7))
@@
   (segment (start 149.86 89.916) (end 152.019 89.916) (width 0.4) (layer F.Cu) (net 7))
   (segment (start 149.098 90.678) (end 149.86 89.916) (width 0.4) (layer F.Cu) (net 7))
-  (segment (start 150.622 99.79) (end 150.146 99.79) (width 0.4) (layer F.Cu) (net 7))
-  (segment (start 150.146 99.79) (end 149.098 100.838) (width 0.4) (layer F.Cu) (net 7))
   (segment (start 149.098 100.838) (end 149.098 107.315) (width 0.4) (layer F.Cu) (net 7))
   (segment (start 149.098 107.315) (end 149.479 107.696) (width 0.4) (layer F.Cu) (net 7))
@@
   (segment (start 189.992 94.64802) (end 181.52302 94.64802) (width 2) (layer B.Cu) (net 10))
   (segment (start 181.52302 94.64802) (end 180.57 93.695) (width 2) (layer B.Cu) (net 10))
-  (segment (start 152.842 107.696) (end 153.416 107.696) (width 0.4) (layer F.Cu) (net 11))
-  (segment (start 152.654 99.822) (end 154.178 98.298) (width 0.4) (layer F.Cu) (net 11))
-  (segment (start 152.654 102.108) (end 152.654 99.822) (width 0.4) (layer F.Cu) (net 11))
-  (segment (start 154.432 103.886) (end 152.654 102.108) (width 0.4) (layer F.Cu) (net 11))
-  (segment (start 154.432 106.68) (end 154.432 103.886) (width 0.4) (layer F.Cu) (net 11))
-  (segment (start 153.416 107.696) (end 154.432 106.68) (width 0.4) (layer F.Cu) (net 11))
+  (segment (start 152.842 107.696) (end 152.7556 107.696) (width 0.254) (layer F.Cu) (net 11) (status C00000))
+  (segment (start 152.7556 107.696) (end 152.146 107.0864) (width 0.254) (layer F.Cu) (net 11) (status 400000))
+  (segment (start 152.146 107.0864) (end 152.146 103.5812) (width 0.254) (layer F.Cu) (net 11))
+  (segment (start 152.146 103.5812) (end 151.6888 103.124) (width 0.254) (layer F.Cu) (net 11))
+  (segment (start 151.6888 103.124) (end 151.6888 102.9716) (width 0.254) (layer F.Cu) (net 11))
+  (via (at 151.6888 102.9716) (size 0.6858) (drill 0.3302) (layers F.Cu B.Cu) (net 11))
+  (segment (start 151.6888 102.9716) (end 152.4508 102.2096) (width 0.254) (layer B.Cu) (net 11))
+  (segment (start 152.4508 102.2096) (end 152.4508 100.0252) (width 0.254) (layer B.Cu) (net 11))
+  (segment (start 152.4508 100.0252) (end 154.178 98.298) (width 0.254) (layer B.Cu) (net 11) (status 800000))
   (segment (start 157.414 104.14) (end 160.274 104.14) (width 0.4) (layer F.Cu) (net 12))
   (segment (start 161.798 102.616) (end 161.798 100.838) (width 0.4) (layer F.Cu) (net 12))

Commit message: logo movido
Parts:
- moved G*** 0.14 mm to (152.4, 106.6)
Changed lines of the file:
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@@
   )
   (module Grape:atom_small (layer B.Cu)
-    (at 152.3365 106.426 90)
+    (at 152.4 106.553 90)
     (fp_text reference G*** (at 0 0 90) (layer B.SilkS) hide
       (effects (font (thickness 0.3)) (justify mirror))
@@
   (segment (start 150.942 91.882) (end 150.792 92.032) (width 0.3) (layer F.Cu) (net 1))
   (segment (start 150.792 92.032) (end 150.792 93.726) (width 0.4) (layer F.Cu) (net 1))
-  (segment (start 155.514 106.188) (end 155.3116 106.188) (width 0.254) (layer F.Cu) (net 2) (status C00000))
-  (segment (start 155.3116 106.188) (end 154.5336 105.41) (width 0.254) (layer F.Cu) (net 2) (status 400000))
+  (segment (start 155.514 106.188) (end 155.3116 106.188) (width 0.254) (layer F.Cu) (net 2))
+  (segment (start 155.3116 106.188) (end 154.5336 105.41) (width 0.254) (layer F.Cu) (net 2))
   (segment (start 154.5336 105.41) (end 154.5336 104.0892) (width 0.254) (layer F.Cu) (net 2))
   (segment (start 154.5336 104.0892) (end 152.9588 102.5144) (width 0.254) (layer F.Cu) (net 2))
@@
   (segment (start 152.5524 102.5144) (end 152.3492 102.3112) (width 0.254) (layer F.Cu) (net 2))
   (segment (start 152.3492 102.3112) (end 152.3492 98.806) (width 0.254) (layer F.Cu) (net 2))
-  (segment (start 152.3492 98.806) (end 151.1808 97.6376) (width 0.254) (layer F.Cu) (net 2) (status 800000))
-  (segment (start 151.1808 97.6376) (end 150.622 97.6376) (width 0.254) (layer F.Cu) (net 2) (status C00000))
+  (segment (start 152.3492 98.806) (end 151.1808 97.6376) (width 0.254) (layer F.Cu) (net 2))
+  (segment (start 151.1808 97.6376) (end 150.622 97.6376) (width 0.254) (layer F.Cu) (net 2))
   (segment (start 154.178 100.838) (end 154.178 102.87) (width 0.5) (layer B.Cu) (net 3))
   (segment (start 153.246 104.31) (end 153.246 105.41) (width 0.5) (layer F.Cu) (net 3))
@@
   (segment (start 189.992 94.64802) (end 181.52302 94.64802) (width 2) (layer B.Cu) (net 10))
   (segment (start 181.52302 94.64802) (end 180.57 93.695) (width 2) (layer B.Cu) (net 10))
-  (segment (start 152.842 107.696) (end 152.7556 107.696) (width 0.254) (layer F.Cu) (net 11) (status C00000))
-  (segment (start 152.7556 107.696) (end 152.146 107.0864) (width 0.254) (layer F.Cu) (net 11) (status 400000))
+  (segment (start 152.842 107.696) (end 152.7556 107.696) (width 0.254) (layer F.Cu) (net 11))
+  (segment (start 152.7556 107.696) (end 152.146 107.0864) (width 0.254) (layer F.Cu) (net 11))
   (segment (start 152.146 107.0864) (end 152.146 103.5812) (width 0.254) (layer F.Cu) (net 11))
   (segment (start 152.146 103.5812) (end 151.6888 103.124) (width 0.254) (layer F.Cu) (net 11))
@@
   (segment (start 151.6888 102.9716) (end 152.4508 102.2096) (width 0.254) (layer B.Cu) (net 11))
   (segment (start 152.4508 102.2096) (end 152.4508 100.0252) (width 0.254) (layer B.Cu) (net 11))
-  (segment (start 152.4508 100.0252) (end 154.178 98.298) (width 0.254) (layer B.Cu) (net 11) (status 800000))
+  (segment (start 152.4508 100.0252) (end 154.178 98.298) (width 0.254) (layer B.Cu) (net 11))
   (segment (start 157.414 104.14) (end 160.274 104.14) (width 0.4) (layer F.Cu) (net 12))
   (segment (start 161.798 102.616) (end 161.798 100.838) (width 0.4) (layer F.Cu) (net 12))
